File: HDK/SmallGeneral.kicad_pcb (KiCad board)
At the start: 2 copper layers, 80 x 50 mm, 51 parts, among them J101 USB_C, SW101 SW_Push, SW102 SW_Push, SW103 SW_Push, U101 STM32F072CBTx, U102 TJA1042T-3, U103 AMS1117-3.3, U104 AMS1117-5.0

Commit message: updated rev4
Parts:
- U101: value STM32F072CBTx -> STM32F072CBT6
Connections:
- SG101 pad E1: unconnected-(SG101B-5V-PadE1) -> +5V
- SG101 pad E2: unconnected-(SG101B-3V3-PadE2) -> +3V3
- SG101 pad E3: /SPI_MISO -> /SPI_IRQ
- SG101 pad E5: GND -> /SPI_SCLK
- SG101 pad E6: +5V -> /SPI_MISO
- SG101 pad E7: +3V3 -> /SPI_MOSI
- SG101 pad E8: /SPI_SCLK -> /SPI_CS
Changed lines of the file:
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@@
 		(allow_soldermask_bridges_in_footprints no)
 		(pcbplotparams
-			(layerselection 0x0001030_ffffffff)
+			(layerselection 0x00010ff_ffffffff)
 			(plot_on_all_layers_selection 0x0001000_00000000)
 			(disableapertmacros no)
@@
 			(sketchpadsonfab no)
 			(subtractmaskfromsilk no)
-			(outputformat 4)
+			(outputformat 1)
 			(mirror no)
 			(drillshape 0)
 			(scaleselection 1)
-			(outputdirectory "../Renders/R4/")
+			(outputdirectory "../Production/v4/small-general-prod/")
 		)
 	)
@@
 	(net 62 "unconnected-(J101-SHIELD-PadS1)_1")
 	(net 63 "unconnected-(J101-SHIELD-PadS1)_2")
-	(net 64 "unconnected-(SG101B-5V-PadE1)")
-	(net 65 "unconnected-(SG101B-3V3-PadE2)")
 	(footprint "Capacitor_SMD:C_0805_2012Metric"
 		(layer "F.Cu")
@@
 			)
 		)
-		(property "Value" "STM32F072CBTx"
+		(property "Value" "STM32F072CBT6"
 			(at 0 5.85 0)
 			(layer "F.Fab")
@@
 			(remove_unused_layers no)
 			(roundrect_rratio 0.208333)
-			(net 64 "unconnected-(SG101B-5V-PadE1)")
+			(net 3 "+5V")
 			(pinfunction "5V")
 			(pintype "input")
@@
 			(layers "*.Cu" "*.Mask")
 			(remove_unused_layers no)
-			(net 65 "unconnected-(SG101B-3V3-PadE2)")
+			(net 1 "+3V3")
 			(pinfunction "3V3")
 			(pintype "input")
@@
 			(layers "*.Cu" "*.Mask")
 			(remove_unused_layers no)
-			(net 31 "/SPI_MISO")
+			(net 32 "/SPI_IRQ")
 			(pinfunction "SPI_IRQ")
 			(pintype "input")
@@
 			(layers "*.Cu" "*.Mask")
 			(remove_unused_layers no)
-			(net 2 "GND")
+			(net 30 "/SPI_SCLK")
 			(pinfunction "SPI_SCLK")
 			(pintype "input")
@@
 			(layers "*.Cu" "*.Mask")
 			(remove_unused_layers no)
-			(net 3 "+5V")
+			(net 31 "/SPI_MISO")
 			(pinfunction "SPI_MISO")
 			(pintype "input")
@@
 			(layers "*.Cu" "*.Mask")
 			(remove_unused_layers no)
-			(net 1 "+3V3")
+			(net 33 "/SPI_MOSI")
 			(pinfunction "SPI_MOSI")
 			(pintype "input")
@@
 			(layers "*.Cu" "*.Mask")
 			(remove_unused_layers no)
-			(net 30 "/SPI_SCLK")
+			(net 34 "/SPI_CS")
 			(pinfunction "SPI_CS")
 			(pintype "input")
@@
 			)
 		)
-		(property "LCSC" "C25804"
+		(property "LCSC" " C21190"
 			(at 0 0 0)
 			(layer "F.Fab")
@@
 			)
 		)
-		(property "LCSC" "C25804"
+		(property "LCSC" " C21190"
 			(at 0 0 0)
 			(layer "F.Fab")

Commit message: updated rev4.1
Parts:
- added JP101: Jumper_2_Open, Connector_PinHeader_2.54mm:PinHeader_1x02_P2.54mm_Vertical, F.Cu at (169.2, 125.9)
- R105, R106, R107: value 200 -> 300
Connections:
- SG101 pad L5: (no net) -> VCC
- SG101 pad L6: (no net) -> GND
Routing:
- net +5V: track 154.3 -> 166.1 mm
- net VCC: track 124.1 -> 134.2 mm
- net VBUS: track 14.6 -> 20.9 mm
Other:
- board text added: "JLCJLCJLCJLC"
- board text added: "Rev4.1"
- board text removed: "Rev4"
